File: hardware/IPiMI/iPiMI.sch (KiCad schematic (older format))
At the start: 15 parts, among them J1 Conn_02x10_Odd_Even, J2 Conn_01x06, J3 Conn_02x10_Odd_Even, SW1 SW_Push, SW2 SW_Push, U1 PC817, U2 PC817, U3 PC817, U4 PC817

Commit message: added images
Other:
- note added: "12/28/2021"
- note added: "IPiMI"
- note added: "Version 1.0"
- moved on the sheet: D1, D2, J1, J2, J3, R1, R2, R5, R6, SW1, SW2, U1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
